Commit message: visual and collision working

File: description/robot_core.xacro (robot description, xacro)
@@ -14,4 +14,7 @@
         <color rgba="0 0 1 1"/>
     </material>
+    <material name="yellow">
+        <color rgba="1 1 0 1"/>
+    </material>
     <material name="black">
         <color rgba="0 0 0 1"/>
@@ -24,29 +27,55 @@
         <parent link="base_link"/>
         <child link="chassis"/>
-        <origin xyz="-0.043 0 0"/>
+        <origin xyz="-0.02115 0 0.01125"/>
     </joint>
     <link name="chassis">
+        <!-- Main chassis box -->
         <visual>
-            <origin xyz="0.07 0 0.075"/>
+            <origin xyz="0.0695 0 0.03425"/>
             <geometry>
-                <box size="0.140 0.1 0.15"/>
+                <box size="0.139 0.099 0.0685"/>
             </geometry>
-            <material name="white"/>
+            <material name="grey"/>
         </visual>
         <collision>
-            <origin xyz="0.07 0 0.075"/>
+            <origin xyz="0.0695 0 0.03425"/>
             <geometry>
-                <box size="0.140 0.1 0.15"/>
+                <box size="0.139 0.099 0.0685"/>
             </geometry>
         </collision>
-        <xacro:inertial_box mass="0.5" x="0.14" y="0.1" z="0.15">
-            <origin xyz="0.07 0 0.075" rpy="0 0 0"/>
-        </xacro:inertial_box>
+        <!-- Raspberry pi box-->
+        <visual>
+            <origin xyz="0.067 0 0.0871"/>
+            <geometry>
+                <box size="0.056 0.085 0.0372"/>
+            </geometry>
+            <material name="grey"/>
+        </visual>
+        <collision>
+            <origin xyz="0.067 0 0.0871"/>
+            <geometry>
+                <box size="0.056 0.085 0.0372"/>
+            </geometry>
+        </collision>
+        <!-- Caster wheel box -->
+        <visual>
+            <origin xyz="0.1315 0 -0.02"/>
+            <geometry>
+                <box size="0.015 0.05 0.04"/>
+            </geometry>
+            <material name="grey"/>
+        </visual>
+        <collision>
+            <origin xyz="0.1315 0 -0.02"/>
+            <geometry>
+                <box size="0.015 0.05 0.04"/>
+            </geometry>
+        </collision>
     </link>
-    <!-- LEFT WHEEL LINK -->
+    <!-- LEFT WHEEL LINK-->
     <joint name="left_wheel_joint" type="continuous">
         <parent link="base_link"/>
         <child link="left_wheel"/>
-        <origin xyz="0 0.07 0" rpy="-${pi/2} 0 0"/>
+        <origin xyz="0 0.062 0" rpy="-${pi/2} 0 0"/>
         <axis xyz="0 0 1"/>
     </joint>
@@ -56,5 +85,5 @@
                 <cylinder radius="0.0325" length="0.025"/>
             </geometry>
-            <material name="blue"/>
+            <material name="yellow"/>
         </visual>
         <collision>
@@ -63,13 +92,10 @@
             </geometry>
         </collision>
-        <xacro:inertial_cylinder mass="0.1" length="0.025" radius="0.0325">
-            <origin xyz="0 0 0" rpy="0 0 0"/>
-        </xacro:inertial_cylinder>
     </link>
-    <!-- RIGHT WHEEL LINK -->
+    <!-- RIGHT WHEEL LINK-->
     <joint name="right_wheel_joint" type="continuous">
         <parent link="base_link"/>
         <child link="right_wheel"/>
-        <origin xyz="0 -0.07 0" rpy="${pi/2} 0 0"/>
+        <origin xyz="0 -0.062 0" rpy="${pi/2} 0 0"/>
         <axis xyz="0 0 -1"/>
     </joint>
@@ -79,5 +105,5 @@
                 <cylinder radius="0.0325" length="0.025"/>
             </geometry>
-            <material name="blue"/>
+            <material name="yellow"/>
         </visual>
         <collision>
@@ -86,29 +112,23 @@
             </geometry>
         </collision>
-        <xacro:inertial_cylinder mass="0.1" length="0.025" radius="0.0325">
-            <origin xyz="0 0 0" rpy="0 0 0"/>
-        </xacro:inertial_cylinder>
     </link>
-    <!-- CARSTER WHEEL LINK -->
+    <!-- CASTER WHEEL LINK -->
     <joint name="caster_wheel_joint" type="fixed">
         <parent link="chassis"/>
         <child link="caster_wheel"/>
-        <origin xyz="0.1 0 0"/>
+        <origin xyz="0.1315 0 -0.03625"/>
     </joint>
     <link name="caster_wheel">
         <visual>
             <geometry>
-                <sphere radius="0.0325"/>
+                <sphere radius="0.0075"/>
             </geometry>
-            <material name="black"/>
+            <material name="white"/>
         </visual>
         <collision>
             <geometry>
-                <sphere radius="0.0325"/>
+                <sphere radius="0.0075"/>
             </geometry>
         </collision>
-        <xacro:inertial_sphere mass="0.1" radius="0.0325">
-            <origin xyz="0 0 0" rpy="0 0 0"/>
-        </xacro:inertial_sphere>
     </link>
 </robot>

Commit message: adding inertias

File: description/robot_core.xacro (robot description, xacro)
@@ -72,4 +72,7 @@
             </geometry>
         </collision>
+        <xacro:inertial_box mass="0.95968" x="0.139" y="0.099" z="0.0685">
+            <origin xyz="0.0695 0 0.03425" rpy="0 0 0"/>
+        </xacro:inertial_box>
     </link>
     <!-- LEFT WHEEL LINK-->
@@ -92,4 +95,7 @@
             </geometry>
         </collision>
+        <xacro:inertial_cylinder mass="0.0257" length="0.025" radius="0.0325">
+            <origin xyz="0 0 0" rpy="0 0 0"/>
+        </xacro:inertial_cylinder>
     </link>
     <!-- RIGHT WHEEL LINK-->
@@ -112,4 +118,7 @@
             </geometry>
         </collision>
+        <xacro:inertial_cylinder mass="0.0257" length="0.025" radius="0.0325">
+            <origin xyz="0 0 0" rpy="0 0 0"/>
+        </xacro:inertial_cylinder>
     </link>
     <!-- CASTER WHEEL LINK -->
@@ -131,4 +140,7 @@
             </geometry>
         </collision>
+        <xacro:inertial_sphere mass="0.01382" radius="0.0075">
+            <origin xyz="0 0 0" rpy="0 0 0"/>
+        </xacro:inertial_sphere>
     </link>
 </robot>

Commit message: Adding launch file for gazebo and modifying the bot colors

File: description/robot_core.xacro (robot description, xacro)
@@ -36,5 +36,5 @@
                 <box size="0.139 0.099 0.0685"/>
             </geometry>
-            <material name="grey"/>
+            <material name="blue"/>
         </visual>
         <collision>
@@ -50,5 +50,5 @@
                 <box size="0.056 0.085 0.0372"/>
             </geometry>
-            <material name="grey"/>
+            <material name="blue"/>
         </visual>
         <collision>
@@ -64,5 +64,5 @@
                 <box size="0.015 0.05 0.04"/>
             </geometry>
-            <material name="grey"/>
+            <material name="blue"/>
         </visual>
         <collision>
@@ -76,4 +76,7 @@
         </xacro:inertial_box>
     </link>
+    <gazebo reference="chassis">
+        <material>Gazebo/Blue</material>
+    </gazebo>
     <!-- LEFT WHEEL LINK-->
     <joint name="left_wheel_joint" type="continuous">
@@ -99,4 +102,7 @@
         </xacro:inertial_cylinder>
     </link>
+    <gazebo reference="left_wheel">
+        <material>Gazebo/Yellow</material>
+    </gazebo>
     <!-- RIGHT WHEEL LINK-->
     <joint name="right_wheel_joint" type="continuous">
@@ -122,4 +128,7 @@
         </xacro:inertial_cylinder>
     </link>
+    <gazebo reference="right_wheel">
+        <material>Gazebo/Yellow</material>
+    </gazebo>
     <!-- CASTER WHEEL LINK -->
     <joint name="caster_wheel_joint" type="fixed">
@@ -144,3 +153,6 @@
         </xacro:inertial_sphere>
     </link>
+    <gazebo reference="caster_wheel">
+        <material>Gazebo/White</material>
+    </gazebo>
 </robot>

Commit message: adding lidar files, working with gazebo

File: description/robot_core.xacro (robot description, xacro)
@@ -19,4 +19,7 @@
     <material name="black">
         <color rgba="0 0 0 1"/>
+    </material>
+    <material name="red">
+        <color rgba="1 0 0 1"/>
     </material>
     <!-- BASE LINK -->

Commit message: adding files for slam toolbox and adding lidar to robot launch file

File: description/robot_core.xacro (robot description, xacro)
@@ -25,4 +25,12 @@
     <!-- BASE LINK -->
     <link name="base_link">
+    </link>
+    <!-- BASE FOOTPRINT LINK -->
+    <joint name="base_footprint_joint" type="fixed">
+        <parent link="base_link"/>
+        <child link="base_footprint"/>
+        <origin xyz="0 0 0" rpy="0 0 0"/>
+    </joint>
+    <link name="base_footprint">
     </link>
     <!-- CHASSIS LINK -->
