Commit message: ros2 control working with gazebo

File: description/depth_camera.xacro (robot description, xacro)
@@ -4,10 +4,10 @@
         <parent link="chassis"/>
         <child link="camera_link"/>
-        <origin xyz="0.305 0 0.08" rpy="0 0 0"/>
+        <origin xyz="0.130 0 0.081" rpy="0 0 0"/>
     </joint>
     <link name="camera_link">
         <visual>
             <geometry>
-                <box size="0.010 0.03 0.03"/>
+                <box size="0.025 0.09 0.025"/>
             </geometry>
             <material name="red"/>

File: description/ros2_control.xacro (robot description, xacro)
@@ -1,5 +1,29 @@
 <?xml version="1.0"?>
 <robot xmlns:xacro="http://www.ros.org/wiki/xacro"  name="robot">
-   <ros2_control>
+   <ros2_control name="GazeboSystem" type="system">
+      <hardware>
+         <plugin>gazebo_ros2_control/GazeboSystem</plugin>
+      </hardware>
+      <joint name="left_wheel_joint">
+         <command_interface name="velocity">
+            <param name="min">-10</param>
+            <param name="max">10</param>
+         </command_interface>
+         <state_interface name="velocity"/>
+         <state_interface name="position"/>
+      </joint>
+      <joint name="right_wheel_joint">
+         <command_interface name="velocity">
+            <param name="min">-10</param>
+            <param name="max">10</param>
+         </command_interface>
+         <state_interface name="velocity"/>
+         <state_interface name="position"/>
+      </joint>
    </ros2_control>
+   <gazebo>
+        <plugin name="gazebo_ros2_control" filename="libgazebo_ros2_control.so">
+            <parameters>$(find my_bot)/config/my_controllers.yaml</parameters>
+        </plugin>
+    </gazebo>
 </robot>

Commit message: adding depth camera description and launchfile

File: description/depth_camera.xacro (robot description, xacro)
@@ -1,4 +1,5 @@
 <?xml version="1.0"?>
-<robot xmlns:xacro="http://www.ros.org/wiki/xacro" >
+<robot xmlns:xacro="http://www.ros.org/wiki/xacro">
+    <!-- Mounting RealSense D435 to the chassis -->
     <joint name="camera_joint" type="fixed">
         <parent link="chassis"/>
@@ -6,4 +7,5 @@
         <origin xyz="0.130 0 0.081" rpy="0 0 0"/>
     </joint>
+    <!-- Base Link of RealSense D435 -->
     <link name="camera_link">
         <visual>
@@ -14,14 +16,23 @@
         </visual>
     </link>
-    <joint name="camera_optical_joint" type="fixed">
+    <!-- Depth Optical Frame -->
+    <joint name="camera_depth_optical_joint" type="fixed">
         <parent link="camera_link"/>
-        <child link="camera_link_optical"/>
+        <child link="camera_depth_optical_frame"/>
         <origin xyz="0 0 0" rpy="${-pi/2} 0 ${-pi/2}"/>
     </joint>
-    <link name="camera_link_optical"></link>
+    <link name="camera_depth_optical_frame"/>
+    <!-- Color Optical Frame -->
+    <joint name="camera_color_optical_joint" type="fixed">
+        <parent link="camera_link"/>
+        <child link="camera_color_frame"/>
+        <origin xyz="0 0 0" rpy="0 0 0"/>
+    </joint>
+    <link name="camera_color_frame"/>
+    <!-- Gazebo Simulation Settings -->
     <gazebo reference="camera_link">
         <material>Gazebo/Red</material>
-        <sensor name="camera" type="depth">
-            <pose> 0 0 0 0 0 0 </pose>
+        <sensor name="depth_camera" type="depth">
+            <pose>0 0 0 0 0 0</pose>
             <visualize>true</visualize>
             <update_rate>10</update_rate>
@@ -39,5 +50,5 @@
             </camera>
             <plugin name="camera_controller" filename="libgazebo_ros_camera.so">
-                <frame_name>camera_link_optical</frame_name>
+                <frame_name>camera_depth_optical_frame</frame_name>
                 <min_depth>0.1</min_depth>
                 <max_depth>100.0</max_depth>
